File: _autosave-dream_controller.kicad_pcb (KiCad board)
At the start: 2 copper layers, 40 parts, among them J1 USB_B_Micro, Q1 Q_NMOS_DGS, Q2 Q_NMOS_DGS, Q3 Q_NMOS_DGS, Q4 Q_NMOS_DGS, SW1 SW_Push, U1 RP2040, U2 W25Q32JVSS, U3 MAX4073TAUT, U4 DRV8770RGER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

Commit message: continued CANification
Parts:
- moved C2 17.7 mm to (108.6, 122.6)
Changed lines of the file:
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@@
   )
   (footprint "Capacitor_SMD:C_0603_1608Metric" (layer "F.Cu")
-    (at 91.44 126.97)
+    (at 108.585 122.555)
     (descr "Capacitor SMD 0603 (1608 Metric), square (rectangular) end terminal, IPC_7351 nominal, (Body size source: IPC-SM-782 page 76, https://www.pcb-3d.com/wordpress/wp-content/uploads/ipc-sm-782a_amendment_1_and_2.pdf), generated with kicad-footprint-generator")
     (tags "capacitor")
