File: driver.kicad_sch (KiCad schematic)
At the start: 6 parts, among them Q1 Q_NMOS_DGS, Q2 Q_NMOS_DGS, Q3 Q_NMOS_DGS, Q4 Q_NMOS_DGS

Commit message: finished schematic design
Parts:
- added C?: 0.1u, symbol Device:C
- added C? (x2): 100n, symbol Device:C
- added J?: MOTOR, symbol Connector:Conn_01x02_Female
- added J?: TEST POINTS, symbol Connector:Conn_01x05_Male
- added R1: 0.3m, symbol Device:R_US
- added U?: MAX4073TAUT, symbol CURRENT_AMP:MAX4073TAUT
Connections:
- net GND: now also U?.25 (EPAD), C?.1, U?.1 (GND), U?.2 (GND)
- net INHA: now also J?.1 (Pin_1)
- net INHB: now also J?.3 (Pin_3)
- net INLA: now also J?.2 (Pin_2)
- net INLB: now also J?.4 (Pin_4)
- net M_A: now also J?.2 (Pin_2)
- net M_B: now also J?.1 (Pin_1)
- net VCC: now also C?.2, C?.2, R1.1, U?.4 (RS+); no longer C16.2, Q1.1 (D), Q2.1 (D), U?.4 (GVDD)
- net at U?.17 (BSTB): now also C?.1
- net at U?.20 (BSTA): now also C?.1
- new net +15V: C16.2, U?.4 (GVDD)
- new net +3V3: C?.2, U?.3 (VCC)
- new net CURRENT: J?.5 (Pin_5), U?.6 (OUT)
- new net RS-: Q1.1 (D), Q2.1 (D), R1.2, U?.5 (RS-)
- no-connect marks 0 -> 5
Other:
- moved on the sheet: Q1, Q2, Q3, Q4

Commit message: assigned footprints and started PCB
Parts:
- C16: footprint (none) -> Capacitor_SMD:C_0603_1608Metric
- C18, C19, C20: renamed from C?; footprint (none) -> Capacitor_SMD:C_0603_1608Metric
- Q1, Q2, Q3, Q4: footprint (none) -> MOSFET:PowerPAK_SO-8_FET
- R4: renamed from R1; footprint (none) -> Resistor_SMD:R_2512_6332Metric
- U3: renamed from U?; footprint (none) -> Package_TO_SOT_SMD:TSOT-23-6_HandSoldering
- U4: renamed from U?; footprint VQFN24_RGE_TEX -> DRIVER:DRV8770RGER
- gave numbers to parts that had none: 2
Changed lines of the file:
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@@
       (effects (font (size 1.27 1.27)) (justify left))
     )
-    (property "Footprint" "" (id 2) (at 154.94 59.69 0)
+    (property "Footprint" "MOSFET:PowerPAK_SO-8_FET" (id 2) (at 154.94 59.69 0)
       (effects (font (size 1.27 1.27)) hide)
     )
@@
     (property "Reference" "C16" (id 0) (at 54.61 60.96 90))
     (property "Value" "10uF" (id 1) (at 54.61 63.5 90))
-    (property "Footprint" "" (id 2) (at 58.42 67.6148 0)
+    (property "Footprint" "Capacitor_SMD:C_0603_1608Metric" (id 2) (at 58.42 67.6148 0)
       (effects (font (size 1.27 1.27)) hide)
     )
@@
   (symbol (lib_id "DRIVER:DRV8770RGER") (at 68.58 60.96 0) (unit 1)
     (in_bom yes) (on_board yes) (fields_autoplaced)
-    (property "Reference" "U?" (id 0) (at 91.44 49.53 0)
+    (property "Reference" "U4" (id 0) (at 91.44 49.53 0)
       (effects (font (size 1.524 1.524)))
     )
@@
       (effects (font (size 1.524 1.524)))
     )
-    (property "Footprint" "VQFN24_RGE_TEX" (id 2) (at 91.44 54.864 0)
+    (property "Footprint" "DRIVER:DRV8770RGER" (id 2) (at 91.44 54.864 0)
       (effects (font (size 1.524 1.524)) hide)
     )
@@
   (symbol (lib_id "power:VCC") (at 170.18 43.18 0) (unit 1)
     (in_bom yes) (on_board yes) (fields_autoplaced)
-    (property "Reference" "#PWR?" (id 0) (at 170.18 46.99 0)
+    (property "Reference" "#PWR0129" (id 0) (at 170.18 46.99 0)
       (effects (font (size 1.27 1.27)) hide)
     )
@@
   (symbol (lib_id "power:GND") (at 120.65 60.96 90) (unit 1)
     (in_bom yes) (on_board yes) (fields_autoplaced)
-    (property "Reference" "#PWR?" (id 0) (at 127 60.96 0)
+    (property "Reference" "#PWR0125" (id 0) (at 127 60.96 0)
       (effects (font (size 1.27 1.27)) hide)
     )
@@
   (symbol (lib_id "power:+15V") (at 58.42 58.42 0) (unit 1)
     (in_bom yes) (on_board yes) (fields_autoplaced)
-    (property "Reference" "#PWR?" (id 0) (at 58.42 62.23 0)
+    (property "Reference" "#PWR0124" (id 0) (at 58.42 62.23 0)
       (effects (font (size 1.27 1.27)) hide)
     )
@@
   (symbol (lib_id "power:GND") (at 50.8 73.66 0) (unit 1)
     (in_bom yes) (on_board yes)
-    (property "Reference" "#PWR?" (id 0) (at 50.8 80.01 0)
+    (property "Reference" "#PWR0123" (id 0) (at 50.8 80.01 0)
       (effects (font (size 1.27 1.27)) hide)
     )
@@
   (symbol (lib_id "Device:R_US") (at 170.18 49.53 0) (unit 1)
     (in_bom yes) (on_board yes) (fields_autoplaced)
-    (property "Reference" "R1" (id 0) (at 172.72 48.2599 0)
+    (property "Reference" "R4" (id 0) (at 172.72 48.2599 0)
       (effects (font (size 1.27 1.27)) (justify left))
     )
@@
       (effects (font (size 1.27 1.27)) (justify left))
     )
-    (property "Footprint" "" (id 2) (at 171.196 49.784 90)
+    (property "Footprint" "Resistor_SMD:R_2512_6332Metric" (id 2) (at 171.196 49.784 90)
       (effects (font (size 1.27 1.27)) hide)
     )
@@
   (symbol (lib_id "power:GND") (at 59.69 88.9 270) (unit 1)
     (in_bom yes) (on_board yes)
-    (property "Reference" "#PWR?" (id 0) (at 53.34 88.9 0)
+    (property "Reference" "#PWR0122" (id 0) (at 53.34 88.9 0)
       (effects (font (size 1.27 1.27)) hide)
     )
@@
   (symbol (lib_id "Device:C") (at 82.55 20.32 90) (unit 1)
     (in_bom yes) (on_board yes)
-    (property "Reference" "C?" (id 0) (at 82.55 13.97 90))
+    (property "Reference" "C18" (id 0) (at 82.55 13.97 90))
     (property "Value" "0.1u" (id 1) (at 82.55 16.51 90))
-    (property "Footprint" "" (id 2) (at 86.36 19.3548 0)
+    (property "Footprint" "Capacitor_SMD:C_0603_1608Metric" (id 2) (at 86.36 19.3548 0)
       (effects (font (size 1.27 1.27)) hide)
     )
@@
   (symbol (lib_id "power:VCC") (at 127 78.74 270) (unit 1)
     (in_bom yes) (on_board yes) (fields_autoplaced)
-    (property "Reference" "#PWR?" (id 0) (at 123.19 78.74 0)
+    (property "Reference" "#PWR0126" (id 0) (at 123.19 78.74 0)
       (effects (font (size 1.27 1.27)) hide)
     )
@@
       (effects (font (size 1.27 1.27)) (justify left))
     )
-    (property "Footprint" "" (id 2) (at 186.69 59.69 0)
+    (property "Footprint" "MOSFET:PowerPAK_SO-8_FET" (id 2) (at 186.69 59.69 0)
       (effects (font (size 1.27 1.27)) hide)
     )
@@
   (symbol (lib_id "Connector:Conn_01x02_Female") (at 172.72 80.01 270) (unit 1)
     (in_bom yes) (on_board yes)
-    (property "Reference" "J?" (id 0) (at 173.99 78.1049 90)
+    (property "Reference" "J4" (id 0) (at 173.99 78.1049 90)
       (effects (font (size 1.27 1.27)) (justify left))
     )
@@
   (symbol (lib_id "power:GND") (at 170.18 92.71 0) (unit 1)
     (in_bom yes) (on_board yes) (fields_autoplaced)
-    (property "Reference" "#PWR?" (id 0) (at 170.18 99.06 0)
+    (property "Reference" "#PWR0128" (id 0) (at 170.18 99.06 0)
       (effects (font (size 1.27 1.27)) hide)
     )
@@
   (symbol (lib_id "power:GND") (at 91.44 40.64 0) (unit 1)
     (in_bom yes) (on_board yes) (fields_autoplaced)
-    (property "Reference" "#PWR?" (id 0) (at 91.44 46.99 0)
+    (property "Reference" "#PWR0130" (id 0) (at 91.44 46.99 0)
       (effects (font (size 1.27 1.27)) hide)
     )
@@
   (symbol (lib_id "Device:C") (at 121.92 81.28 90) (unit 1)
     (in_bom yes) (on_board yes)
-    (property "Reference" "C?" (id 0) (at 119.38 85.09 90))
+    (property "Reference" "C20" (id 0) (at 119.38 85.09 90))
     (property "Value" "100n" (id 1) (at 118.11 80.01 90))
-    (property "Footprint" "" (id 2) (at 125.73 80.3148 0)
+    (property "Footprint" "Capacitor_SMD:C_0603_1608Metric" (id 2) (at 125.73 80.3148 0)
       (effects (font (size 1.27 1.27)) hide)
     )
@@
   (symbol (lib_id "Connector:Conn_01x05_Male") (at 135.89 21.59 270) (unit 1)
     (in_bom yes) (on_board yes) (fields_autoplaced)
-    (property "Reference" "J?" (id 0) (at 135.89 16.51 90))
+    (property "Reference" "J3" (id 0) (at 135.89 16.51 90))
     (property "Value" "TEST POINTS" (id 1) (at 135.89 19.05 90))
     (property "Footprint" "" (id 2) (at 135.89 21.59 0)
@@
   (symbol (lib_id "power:+3V3") (at 91.44 19.05 0) (unit 1)
     (in_bom yes) (on_board yes) (fields_autoplaced)
-    (property "Reference" "#PWR?" (id 0) (at 91.44 22.86 0)
+    (property "Reference" "#PWR0131" (id 0) (at 91.44 22.86 0)
       (effects (font (size 1.27 1.27)) hide)
     )
@@
       (effects (font (size 1.27 1.27)) (justify left))
     )
-    (property "Footprint" "" (id 2) (at 154.94 80.01 0)
+    (property "Footprint" "MOSFET:PowerPAK_SO-8_FET" (id 2) (at 154.94 80.01 0)
       (effects (font (size 1.27 1.27)) hide)
     )
@@
   (symbol (lib_id "power:VCC") (at 127 86.36 270) (unit 1)
     (in_bom yes) (on_board yes) (fields_autoplaced)
-    (property "Reference" "#PWR?" (id 0) (at 123.19 86.36 0)
+    (property "Reference" "#PWR0127" (id 0) (at 123.19 86.36 0)
       (effects (font (size 1.27 1.27)) hide)
     )
@@
       (effects (font (size 1.27 1.27)) (justify left))
     )
-    (property "Footprint" "" (id 2) (at 186.69 80.01 0)
+    (property "Footprint" "MOSFET:PowerPAK_SO-8_FET" (id 2) (at 186.69 80.01 0)
       (effects (font (size 1.27 1.27)) hide)
     )
@@
   (symbol (lib_id "CURRENT_AMP:MAX4073TAUT") (at 91.44 30.48 0) (unit 1)
     (in_bom yes) (on_board yes)
-    (property "Reference" "U?" (id 0) (at 99.06 20.32 0))
+    (property "Reference" "U3" (id 0) (at 99.06 20.32 0))
     (property "Value" "MAX4073TAUT" (id 1) (at 99.06 22.86 0))
-    (property "Footprint" "" (id 2) (at 91.44 25.4 0)
+    (property "Footprint" "Package_TO_SOT_SMD:TSOT-23-6_HandSoldering" (id 2) (at 91.44 25.4 0)
       (effects (font (size 1.27 1.27)) hide)
     )
@@
   (symbol (lib_id "power:GND") (at 76.2 20.32 270) (unit 1)
     (in_bom yes) (on_board yes)
-    (property "Reference" "#PWR?" (id 0) (at 69.85 20.32 0)
+    (property "Reference" "#PWR0132" (id 0) (at 69.85 20.32 0)
       (effects (font (size 1.27 1.27)) hide)
     )
@@
   (symbol (lib_id "Device:C") (at 121.92 73.66 90) (unit 1)
     (in_bom yes) (on_board yes)
-    (property "Reference" "C?" (id 0) (at 119.38 77.47 90))
+    (property "Reference" "C19" (id 0) (at 119.38 77.47 90))
     (property "Value" "100n" (id 1) (at 118.11 72.39 90))
-    (property "Footprint" "" (id 2) (at 125.73 72.6948 0)
-      (effects (font (size 1.27 1.27)) hide)
-    )
+    (property "Footprint" "Capacitor_SMD:C_0603_1608Metric" (id 2) (at 125.73 72.6948 0)
+      (effects (font (size 1.27 1.27)) hide)
+    )

Commit message: updating to CAN
Connections:
- no-connect marks 5 -> 6
Changed lines of the file:
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@@
   (no_connect (at 114.3 88.9))
   (no_connect (at 114.3 63.5))
+  (no_connect (at 68.58 71.12))
   (wire (pts (xy 189.23 87.63) (xy 189.23 90.17))
     (stroke (width 0) (type default) (color 0 0 0 0))
